Commit message: feat: add dual-arm rviz scene modeling workflow

File: src/planning/descriptions/fairino_dualarm_description/urdf/fairino_dualarm.urdf.xacro (robot description, xacro)
@@ -1,4 +1,8 @@
 <?xml version="1.0"?>
 <robot xmlns:xacro="http://www.ros.org/wiki/xacro" name="fairino_dualarm">
+  <xacro:arg name="left_base_xyz" default="0 0.35 0"/>
+  <xacro:arg name="left_base_rpy" default="0 0 0"/>
+  <xacro:arg name="right_base_xyz" default="0 -0.35 0"/>
+  <xacro:arg name="right_base_rpy" default="0 0 3.141592653589793"/>
   <xacro:include filename="$(find fairino_dualarm_description)/urdf/fairino3_v6_macro.xacro"/>
   <link name="world"/>
@@ -11,5 +15,5 @@
   <link name="left_base"/>
   <joint name="world_to_left_base" type="fixed">
-    <origin xyz="0 0.35 0" rpy="0 0 0"/>
+    <origin xyz="$(arg left_base_xyz)" rpy="$(arg left_base_rpy)"/>
     <parent link="world"/>
     <child link="left_base"/>
@@ -17,5 +21,5 @@
   <link name="right_base"/>
   <joint name="world_to_right_base" type="fixed">
-    <origin xyz="0 -0.35 0" rpy="0 0 3.141592653589793"/>
+    <origin xyz="$(arg right_base_xyz)" rpy="$(arg right_base_rpy)"/>
     <parent link="world"/>
     <child link="right_base"/>

Commit message: stabilize dual-camera runtime mode

File: src/planning/descriptions/fairino_dualarm_description/urdf/fairino_dualarm.urdf.xacro (robot description, xacro)
@@ -4,6 +4,52 @@
   <xacro:arg name="left_base_rpy" default="0 0 0"/>
   <xacro:arg name="right_base_xyz" default="0 -0.35 0"/>
-  <xacro:arg name="right_base_rpy" default="0 0 3.141592653589793"/>
+  <xacro:arg name="right_base_rpy" default="0 0 0"/>
   <xacro:include filename="$(find fairino_dualarm_description)/urdf/fairino3_v6_macro.xacro"/>
+  <xacro:macro name="tcp_depth_camera_collision" params="prefix parent xyz rpy">
+    <link name="${prefix}camera_mount">
+      <visual>
+        <origin xyz="0 0 0" rpy="0 0 0"/>
+        <geometry>
+          <box size="0.045 0.030 0.020"/>
+        </geometry>
+        <material name="${prefix}camera_mount_dark">
+          <color rgba="0.08 0.08 0.08 1.0"/>
+        </material>
+      </visual>
+      <collision>
+        <origin xyz="0 0 0" rpy="0 0 0"/>
+        <geometry>
+          <box size="0.050 0.035 0.025"/>
+        </geometry>
+      </collision>
+    </link>
+    <joint name="${prefix}tcp_to_camera_mount" type="fixed">
+      <origin xyz="${xyz}" rpy="${rpy}"/>
+      <parent link="${parent}"/>
+      <child link="${prefix}camera_mount"/>
+    </joint>
+    <link name="${prefix}camera_body">
+      <visual>
+        <origin xyz="0.035 0 0" rpy="0 0 0"/>
+        <geometry>
+          <box size="0.070 0.040 0.035"/>
+        </geometry>
+        <material name="${prefix}camera_body_black">
+          <color rgba="0.02 0.02 0.02 1.0"/>
+        </material>
+      </visual>
+      <collision>
+        <origin xyz="0.035 0 0" rpy="0 0 0"/>
+        <geometry>
+          <box size="0.075 0.045 0.040"/>
+        </geometry>
+      </collision>
+    </link>
+    <joint name="${prefix}camera_mount_to_body" type="fixed">
+      <origin xyz="0.035 0 0" rpy="0 0 0"/>
+      <parent link="${prefix}camera_mount"/>
+      <child link="${prefix}camera_body"/>
+    </joint>
+  </xacro:macro>
   <link name="world"/>
   <link name="table"/>
@@ -27,3 +73,4 @@
   <xacro:fairino3_v6_arm prefix="left_" parent="left_base" xyz="0 0 0" rpy="0 0 0"/>
   <xacro:fairino3_v6_arm prefix="right_" parent="right_base" xyz="0 0 0" rpy="0 0 0"/>
+  <xacro:tcp_depth_camera_collision prefix="right_" parent="right_tcp" xyz="0.00 0.00 0.035" rpy="0 0 0"/>
 </robot>
